File: hardware/stm32f4-sound/stm32f4-sound.kicad_pcb (KiCad board)
At the start: 2 copper layers, 63.5 x 82.5 mm, 7 parts, among them J1 Conn_02x25_Odd_Even, J3 Conn_02x18_Odd_Even, SW1 SW_UP, SW2 SW_DN, SW3 SW_L, SW4 SW_R, U1 SSD1306_128x64

Commit message: Finalize the PCB
Connections:
- J1 pad 11: unconnected-(J1-Pin_11-Pad11) -> /PE6
- J1 pad 17: unconnected-(J1-Pin_17-Pad17) -> /PE0
- J1 pad 19: unconnected-(J1-Pin_19-Pad19) -> /PB8
- J1 pad 31: unconnected-(J1-Pin_31-Pad31) -> /PD3
- J1 pad 33: unconnected-(J1-Pin_33-Pad33) -> /PD1
- J1 pad 4: unconnected-(J1-Pin_4-Pad4) -> +5V
- J1 pad 43: unconnected-(J1-Pin_43-Pad43) -> /PA8
- J1 pad 45: unconnected-(J1-Pin_45-Pad45) -> /PC8
- J1 pad 49: unconnected-(J1-Pin_49-Pad49) -> GND
- J1 pad 50: unconnected-(J1-Pin_50-Pad50) -> GND
- J1 pad 6: unconnected-(J1-Pin_6-Pad6) -> +3V0
- J3 pad 10: unconnected-(J3-Pin_10-Pad10) -> /PC2
- J3 pad 14: unconnected-(J3-Pin_14-Pad14) -> /PA2
- J3 pad 22: unconnected-(J3-Pin_22-Pad22) -> /PB0
- J3 pad 23: unconnected-(J3-Pin_23-Pad23) -> GND
- J3 pad 26: unconnected-(J3-Pin_26-Pad26) -> /PE8
- J3 pad 3: unconnected-(J3-Pin_3-Pad3) -> GND
- J3 pad 30: unconnected-(J3-Pin_30-Pad30) -> /PE12
- J3 pad 32: unconnected-(J3-Pin_32-Pad32) -> /PE14
- J3 pad 33: unconnected-(J3-Pin_33-Pad33) -> /PE15
- J3 pad 36: unconnected-(J3-Pin_36-Pad36) -> /PB12
- SW1 pad 2: unconnected-(SW1-Pad2) -> /PE8
- SW2 pad 2: unconnected-(SW2-Pad2) -> /PC8
- SW3 pad 2: unconnected-(SW3-Pad2) -> /PB12
- SW4 pad 2: unconnected-(SW4-Pad2) -> /PA8
- U1 pad 3: unconnected-(U1-D0-CLK-Pad3) -> /PB0
- U1 pad 4: unconnected-(U1-D1-DIN-Pad4) -> /PB8
- U1 pad 5: unconnected-(U1-RES-Pad5) -> /PC2
- U1 pad 6: unconnected-(U1-DC-Pad6) -> /PA2
- U1 pad 7: unconnected-(U1-CS-Pad7) -> /PE6
Routing:
- net GND: track 0.00 -> 157.3 mm
- net +5V: track 0.00 -> 57.7 mm
- net /PB0: track 0.00 -> 49.8 mm
- net +3V0: track 0.00 -> 48.9 mm
- net /PA2: track 0.00 -> 48.7 mm, vias 0 -> 2
- net /PB8: track 0.00 -> 47.6 mm
- net /PC2: track 0.00 -> 44.6 mm, vias 0 -> 2
- net /PE6: track 0.00 -> 36.5 mm
- net /PE8: track 0.00 -> 34.6 mm
- net /PC8: track 0.00 -> 31.5 mm
- net /PA8: track 0.00 -> 28.2 mm
- net /PB12: track 0.00 -> 20.2 mm
