File: hardware/stm32f4-sound/stm32f4-sound.kicad_sch (KiCad schematic)
At the start: 7 parts, among them J1 Conn_02x25_Odd_Even, J3 Conn_02x18_Odd_Even, SW1 SW_UP, SW2 SW_DN, SW3 SW_L, SW4 SW_R, U1 SSD1306_128x64

Commit message: Finalize the PCB
Connections:
- net +3V0: now also J1.6 (Pin_6)
- net +5V: now also J1.4 (Pin_4)
- net GND: now also J1.49 (Pin_49), J1.50 (Pin_50), J3.23 (Pin_23), J3.3 (Pin_3)
- net PB12: now reaches SW3.2
- net PB12: now also J3.36 (Pin_36)
- net PE6: now reaches J1.11 (Pin_11)
- net PE6: now also U1.7 (CS)
- net PE0: now reaches J1.17 (Pin_17)
- net PB8: now reaches J1.19 (Pin_19)
- net PB8: now also U1.4 (D1-DIN)
- net PD3: now reaches J1.31 (Pin_31)
- net PD1: now reaches J1.33 (Pin_33)
- net PA8: now reaches J1.43 (Pin_43)
- net PA8: now also SW4.2
- net PC8: now reaches J1.45 (Pin_45)
- net PC8: now also SW2.2
- net PC2: now reaches J3.10 (Pin_10)
- net PC2: now also U1.5 (RES)
- net PA2: now reaches J3.14 (Pin_14)
- net PA2: now also U1.6 (DC)
- net PB0: now reaches J3.22 (Pin_22)
- net PB0: now also U1.3 (D0-CLK)
- net PE8: now reaches J3.26 (Pin_26)
- net PE8: now also SW1.2
- net PE12: now reaches J3.30 (Pin_30)
- net PE14: now reaches J3.32 (Pin_32)
- net PE15: now reaches J3.33 (Pin_33)
Other:
- moved on the sheet: SW2, SW3, SW4
